File: hardware/blueair_pro_m/cap_touch.kicad_sch (KiCad schematic)
At the start: 15 parts, among them IC2 SC_04A, Q13 BC857

Commit message: pcb update
Parts:
- removed IC2: SC_04A, symbol pff_ic:SC_04A
- added U1: SC04A, Package_SO:SO-16_3.9x9.9mm_P1.27mm, symbol pff_ic:SC04A
Connections:
- net PB4: now also U1.13 (OUT0)
- net PB5: now also U1.12 (OUT1)
- net PB6: now also U1.11 (OUT2)
- net at C21.1: now also U1.3 (CDC)
- net at C20.2, C21.2, FB2.1: now also U1.1 (Vss)
- net at R66.2: now also U1.5 (CIN1)
- net at R76.2: now also U1.4 (CIN0)
- net at R71.2: now also U1.6 (CIN2)
- net at C20.1: now also U1.2 (CMOD)
- net at FB1.2: now also U1.16 (Vcc)
- no-connect marks 4 -> 2
Other:
- moved on the sheet: C20, C21, FB1, FB2, R63, R64, R65
