File: hardware/cc1101_module/cc1101_module.kicad_sch (KiCad schematic)
At the start: 69 parts, among them J2 Conn_02x06_Odd_Even, J3 Conn_Coaxial, J4 io expand 0, J5 io expand 1, Q1 BC846, U1 MCP23S08-xSS, U2 MCP23S08-xSS

Commit message: pcb update
Parts:
- added C7, C8, C9: 100n, Capacitor_SMD:C_0805_2012Metric_Pad1.18x1.45mm_HandSolder, symbol Device:C
- added JP1, JP2: SolderJumper_2_Open, Jumper:SolderJumper-2_P1.3mm_Open_TrianglePad1.0x1.5mm, symbol Jumper:SolderJumper_2_Open
- added U3: TC1014-xCT, Package_TO_SOT_SMD:SOT-23-5, symbol Regulator_Linear:TC1014-xCT
- J3: footprint Connector_Coaxial:SMA_Samtec_SMA-J-P-X-ST-EM1_EdgeMount -> pff_connectors:SMA-16
Connections:
- net GND: now also C7.2, C8.2, C9.2, U3.2 (GND)
- net VCC: now also C9.1, JP1.1 (A), JP2.1 (A), U3.5 (VOUT); no longer J4.10 (Pin_10), J5.10 (Pin_10)
- new net: C7.1, U3.4 (Bypass)
- new net: J5.10 (Pin_10), JP1.2 (B)
- new net Vin: C8.1, J4.10 (Pin_10), JP2.2 (B), U3.1 (VIN), U3.3 (~{SHDN})
Other:
- moved on the sheet: C1, C2, D1, Q1, R4, R5

Commit message: pcb verified
Changed lines of the file:
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@@
   (junction (at 146.05 132.08) (diameter 0) (color 0 0 0 0)
   )
-  (junction (at 148.59 43.18) (diameter 0) (color 0 0 0 0)
-  )
   (wire (pts (xy 224.79 62.23) (xy 228.6 62.23))
     (stroke (width 0) (type default))
@@
     (stroke (width 0) (type default))
   )
-  (wire (pts (xy 152.4 43.18) (xy 148.59 43.18))
-    (stroke (width 0) (type default))
-  )
   (wire (pts (xy 85.09 120.65) (xy 85.09 123.19))
     (stroke (width 0) (type default))
@@
     (stroke (width 0) (type default))
   )
-  (wire (pts (xy 152.4 43.18) (xy 152.4 46.99))
-    (stroke (width 0) (type default))
-  )
   (wire (pts (xy 85.09 165.1) (xy 85.09 167.64))
     (stroke (width 0) (type default))
@@
     )
   )
-  (symbol (lib_id "power:PWR_FLAG") (at 152.4 46.99 180) (unit 1)
-    (in_bom yes) (on_board yes) (dnp no)
-    (property "Reference" "#FLG01" (at 152.4 48.895 0)
-      (effects (font (size 1.27 1.27)) hide)
-    )
-    (property "Value" "PWR_FLAG" (at 148.59 52.07 0)
-      (effects (font (size 1.27 1.27)) (justify right))
-    )
-    (property "Footprint" "" (at 152.4 46.99 0)
-      (effects (font (size 1.27 1.27)) hide)
-    )
-    (property "Datasheet" "~" (at 152.4 46.99 0)
-      (effects (font (size 1.27 1.27)) hide)
-    )
-    (pin "1")
-    (instances
-      (project "cc1101_module"
-        (path "/fdd6a173-f1ae-4cc3-bad3-1f09e466a34d"
-          (reference "#FLG01") (unit 1)
-        )
-      )
-    )
-  )
   (symbol (lib_id "Device:R") (at 41.91 170.18 180) (unit 1)
     (in_bom yes) (on_board yes) (dnp no) (fields_autoplaced)
@@
       (effects (font (size 1.27 1.27)) hide)
     )
-    (property "Datasheet" "" (at 50.8 25.4 0)
+    (property "Datasheet" "https://www.radiocontrolli.com/media/1327_ebbd998f731c6483c4ee12d998cd3b2991fd4e84.pdf/o/rc-cc1101-spi-smt-434.pdf" (at 50.8 25.4 0)
       (effects (font (size 1.27 1.27)) hide)
     )
