File: hardware/cc1101_module/cc1101_module.kicad_pcb (KiCad board)
At the start: 4 copper layers, 100 x 36 mm, 73 parts, among them J2 Conn_02x06_Odd_Even, J3 Conn_Coaxial, J4 io expand 0, J5 io expand 1, Q1 BC846, U1 MCP23S08-xSS, U2 MCP23S08-xSS

Commit message: pcb update
Parts:
- added C7: 100n, Capacitor_SMD:C_0805_2012Metric_Pad1.18x1.45mm_HandSolder, F.Cu at (167.4, 107.8)
- added C8: 100n, Capacitor_SMD:C_0805_2012Metric_Pad1.18x1.45mm_HandSolder, F.Cu at (167.4, 109.8)
- added C9: 100n, Capacitor_SMD:C_0805_2012Metric_Pad1.18x1.45mm_HandSolder, F.Cu at (167.4, 102.2)
- added JP1: SolderJumper_2_Open, Jumper:SolderJumper-2_P1.3mm_Open_TrianglePad1.0x1.5mm, B.Cu at (185.7, 106.6)
- added JP2: SolderJumper_2_Open, Jumper:SolderJumper-2_P1.3mm_Open_TrianglePad1.0x1.5mm, B.Cu at (159.0, 106.6)
- added U3: TC1014-xCT, Package_TO_SOT_SMD:SOT-23-5, F.Cu at (167.4, 105.0)
- J3: footprint Connector_Coaxial:SMA_Samtec_SMA-J-P-X-ST-EM1_EdgeMount -> pff_connectors:SMA-16
- moved REF** 36.9 mm to (196.0, 132.0)
- moved J4 36.7 mm to (148.8, 113.1)
- moved J5 36.7 mm to (175.6, 113.1)
- moved R10 36.7 mm to (163.8, 114.3)
- moved R17 36.7 mm to (190.2, 118.3)
- moved R18 36.7 mm to (190.2, 114.3)
- moved R23 36.7 mm to (144.1, 124.3)
- moved R24 36.7 mm to (144.1, 122.3)
- moved R25 36.7 mm to (144.1, 126.3)
- moved R26 36.7 mm to (144.1, 128.3)
- moved R27 36.7 mm to (144.1, 114.3)
- moved R28 36.7 mm to (144.1, 116.3)
- moved R29 36.7 mm to (144.1, 118.3)
- moved R30 36.7 mm to (144.1, 120.3)
- moved R36 36.7 mm to (163.8, 112.3)
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Connections:
- J4 pad 10: VCC -> Vin
- J5 pad 10: VCC -> Net-(J5-Pin_10)
Routing:
- net INT_E1: track 0.00 -> 99.1 mm, vias 0 -> 2
- net CS_E: track 0.00 -> 97.6 mm, vias 0 -> 2
- net MISO: track 10.6 -> 96.1 mm, vias 0 -> 2
- net MOSI: track 9.99 -> 94.9 mm
- net CLK: track 11.1 -> 92.4 mm
- net INT_E0: track 0.00 -> 68.1 mm, vias 0 -> 2
- net CS_CC: track 0.00 -> 31.1 mm, vias 0 -> 2
- net Vin: track 0.00 -> 21.0 mm
- net GDO0: track 0.00 -> 14.7 mm, vias 0 -> 2
- net GND: track 51.4 -> 61.9 mm, vias 31 -> 100
- net VCC: track 25.3 -> 29.9 mm, vias 10 -> 13
- net Net-(J5-Pin_10): track 0.00 -> 3.29 mm
- net Net-(U3-Bypass): track 0.00 -> 1.87 mm
- net Net-(D1-K): track 4.66 -> 3.48 mm
- net Net-(J5-Pin_5): track 17.2 -> 16.3 mm
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- added copper zone on B.Cu, net GND

Commit message: pcb verified
Other:
- board text added: "CC1101, 2x8ch expander module rev. 1 https://github.com/rodan/voidvent Petre Rodan 2023"
- board text added: "CS e MOSI MISO CLK gnd Vcc"
- board text added: "GDO2 INT e0 INT e1 CS CC GND Vcc"
- board text added: "e00 e02 e04 e06 gnd"
- board text added: "e01 e03 e05 e07 Vcc"
- board text added: "e10 e12 e14 e16 gnd"
- board text added: "e11 e13 e15 e17 Vcc"
Changed lines of the file:
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@@
     (tags "mounting hole 3.2mm m3 din965")
     (attr exclude_from_pos_files exclude_from_bom)
-    (fp_text reference "REF**" (at 0 -3.8) (layer "F.SilkS")
+    (fp_text reference "REF**" (at 0 -3.8) (layer "F.SilkS") hide
         (effects (font (size 1 1) (thickness 0.15)))
     )
@@
     (tags "mounting hole 3.2mm m3 din965")
     (attr exclude_from_pos_files exclude_from_bom)
-    (fp_text reference "REF**" (at 0 -3.8) (layer "F.SilkS")
+    (fp_text reference "REF**" (at 0 -3.8) (layer "F.SilkS") hide
         (effects (font (size 1 1) (thickness 0.15)))
     )
@@
     (tags "mounting hole 3.2mm m3 din965")
     (attr exclude_from_pos_files exclude_from_bom)
-    (fp_text reference "REF**" (at 0 -3.8) (layer "F.SilkS")
+    (fp_text reference "REF**" (at 0 -3.8) (layer "F.SilkS") hide
         (effects (font (size 1 1) (thickness 0.15)))
     )
@@
     (tags "mounting hole 3.2mm m3 din965")
     (attr exclude_from_pos_files exclude_from_bom)
-    (fp_text reference "REF**" (at 0 -3.8) (layer "F.SilkS")
+    (fp_text reference "REF**" (at 0 -3.8) (layer "F.SilkS") hide
         (effects (font (size 1 1) (thickness 0.15)))
     )
@@
   (gr_rect (start 100 100) (end 200 136)
     (stroke (width 0.15) (type default)) (fill none) (layer "Margin"))
+  (gr_text "e01\n\ne03\n\ne05\n\ne07\n\nVcc" (at 159.3 106.985 90) (layer "B.SilkS")
+    (effects (font (size 0.78 0.78) (thickness 0.15)) (justify left bottom mirror))
+  )
+  (gr_text "CC1101, 2x8ch expander module  rev. 1\nhttps://github.com/rodan/voidvent\nPetre Rodan 2023" (at 134.9504 103.2004 90) (layer "B.SilkS")
+    (effects (font (size 1 1) (thickness 0.15)) (justify left bottom mirror))
+  )
+  (gr_text "e10\n\ne12\n\ne14\n\ne16\n\ngnd" (at 186.1 114.6558 90) (layer "B.SilkS")
+    (effects (font (size 0.78 0.78) (thickness 0.15)) (justify left bottom mirror))
+  )
+  (gr_text "e00\n\ne02\n\ne04\n\ne06\n\ngnd" (at 159.3 114.9352 90) (layer "B.SilkS")
+    (effects (font (size 0.78 0.78) (thickness 0.15)) (justify left bottom mirror))
+  )
+  (gr_text "CS e\n\nMOSI\n\nMISO\n\nCLK\n\ngnd\n\nVcc" (at 114.5542 111.2 180) (layer "B.SilkS")
+    (effects (font (size 0.78 0.78) (thickness 0.15)) (justify left bottom mirror))
+  )
+  (gr_text "GDO2\n\nINT e0\n\nINT e1\n\nCS CC\n\nGND\n\nVcc" (at 105.6642 111.2 180) (layer "B.SilkS")
+    (effects (font (size 0.78 0.78) (thickness 0.15)) (justify left bottom mirror))
+  )
+  (gr_text "e11\n\ne13\n\ne15\n\ne17\n\nVcc" (at 186.1 106.9596 90) (layer "B.SilkS")
+    (effects (font (size 0.78 0.78) (thickness 0.15)) (justify left bottom mirror))
+  )
   (segment (start 149.2093 128.4224) (end 150.7118 128.4224) (width 0.4) (layer "F.Cu") (net 1))
   (segment (start 140.0532 103.6454) (end 140.8392 103.6454) (width 0.25) (layer "F.Cu") (net 1))

Commit message: pcb sent to production
Routing:
- net GND: track 61.9 -> 62.5 mm
